File: KiCad_proj/digitaalilaite.kicad_sch (KiCad schematic)
At the start: 20 parts, among them U1 UA741, U2 UA741, U3 UA741

Commit message: lähetin tehty
Parts:
- added BC547_1: BC547_TO92_0.1A, VAMK_ANA:TO-92, symbol VAMK_ANA:BC547_TO92_0.1A
- added C7: 100NF_50V_CER, VAMK_C_SMD:C1206, symbol VAMK_C_SMD:100NF_50V_CER
- added R14: 100R, VAMK_R_SMD:1206, symbol VAMK_R_SMD:100R
- added R15: 150R, VAMK_R_SMD:1206, symbol VAMK_R_SMD:150R
- added R3, R4, R5, R6: 150k, VAMK_R_SMD:1206, symbol VAMK_R_SMD:150k
- added TM_BLOCK/2P1: TM_BLOCK_2P, VAMK_CON:TM_BLOCK_2P, symbol VAMK_CON:TM_BLOCK_2P
- added U4: UA741, VAMK_IC_SMD:SO8IC, symbol VAMK_IC_SMD:UA741_SO8
Connections:
- net +12V: now also U4.7 (V+)
- net -12V: now also U4.4 (V-)
- net GND: now also POTENTIO_M/1K_LIN1.3, R11.1, R5.2, TM_BLOCK/2P1.2 (Pin_2)
- net at R10.2, U2.6: now also R3.1
- new net: BC547_1.1 (C), R6.1
- new net: C7.1, R5.1, R6.2, U4.2 (-)
- new net: C7.2, R14.1, U4.6
- new net: BC547_1.2 (B), R14.2
- new net: R3.2, R4.2, U4.3 (+)
- new net: R15.1, R4.1, TM_BLOCK/2P1.1 (Pin_1)
- new net: BC547_1.3 (E), R15.2
- no-connect marks 6 -> 8
Other:
- moved on the sheet: LM35CZ1, R1, R10, R11, R12, R13, R2, R7, R8, R9, U1, U2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

Commit message: lähetin ja ohituskonkat tehty
Parts:
- added C8, C9: 100NF_50V_CER, VAMK_C_SMD:C1206, symbol VAMK_C_SMD:100NF_50V_CER
- C1, C2, C3, C4, C5, C6: footprint VAMK_C:C5_0 -> VAMK_C_SMD:C1206; symbol VAMK_C:100NF_50V_CER -> VAMK_C_SMD:100NF_50V_CER; Order Number Elfa 65-736-87 -> 65-776-88; Storing Location 2.4.4.2 -> EC6, SMD station
Connections:
- net +12V: now also C8.2
- net -12V: now also C9.2
- net GND: now also C8.1, C9.1
Other:
- moved on the sheet: C1, C2, C3, C4, C5, C6
