File: KiCad_proj/signaalinlahetin/signaalinlahetin.kicad_sch (KiCad schematic)
At the start: 32 parts, among them U1 UA741, U2 UA741, U3 UA741, U4 UA741

Commit message: vastaanotin tehty kicad ja ltspice, ltspicessä teholähtö
Parts:
- added TM_BLOCK/3P1: TM_BLOCK_3P, VAMK_CON:TM_BLOCK_3P, symbol VAMK_CON:TM_BLOCK_3P
Connections:
- net +12V: now also LM35CZ1.1 (+VS), TM_BLOCK/3P1.1 (Pin_1)
- net -12V: now also TM_BLOCK/3P1.3 (Pin_3)
- net GND: now also TM_BLOCK/3P1.2 (Pin_2)
- net at R10.1, R9.2: no longer R8.2, R9.1
- new net: R8.2, R9.1

Commit message: signaalin lähetin kaikki osat paikoillaan, ei johtoja vedetty vielä
Other:
- note added: "256"
- moved on the sheet: LM35CZ1
Changed lines of the file:
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@@
 		)
 	)
+	(text "256"
+		(exclude_from_sim no)
+		(at 106.426 101.092 0)
+		(effects
+			(font
+				(size 1.27 1.27)
+			)
+		)
+	)
 	(junction
 		(at 82.55 67.31)
@@
 	(wire
 		(pts
-			(xy 40.64 69.85) (xy 63.5 69.85)
+			(xy 45.72 69.85) (xy 63.5 69.85)
 		)
 		(stroke
@@
 	(symbol
 		(lib_id "power:GND")
-		(at 30.48 77.47 0)
+		(at 35.56 77.47 0)
 		(unit 1)
 		(body_style 1)
@@
 		(fields_autoplaced yes)
 		(property "Reference" "#PWR08"
-			(at 30.48 83.82 0)
+			(at 35.56 83.82 0)
 			(hide yes)
 			(show_name no)
@@
 		)
 		(property "Value" "GND"
-			(at 30.48 82.55 0)
+			(at 35.56 82.55 0)
 			(show_name no)
 			(do_not_autoplace no)
@@
 		)
 		(property "Footprint" ""
-			(at 30.48 77.47 0)
+			(at 35.56 77.47 0)
 			(hide yes)
 			(show_name no)
@@
 		)
 		(property "Datasheet" ""
-			(at 30.48 77.47 0)
+			(at 35.56 77.47 0)
 			(hide yes)
 			(show_name no)
@@
 		)
 		(property "Description" "Power symbol creates a global label with name \"GND\" , ground"
-			(at 30.48 77.47 0)
+			(at 35.56 77.47 0)
 			(hide yes)
 			(show_name no)
@@
 	(symbol
 		(lib_id "VAMK_IC:LM35CZ_TO92")
-		(at 30.48 69.85 0)
+		(at 35.56 69.85 0)
 		(unit 1)
 		(body_style 1)
@@
 		(fields_autoplaced yes)
 		(property "Reference" "LM35CZ1"
-			(at 21.59 69.8499 0)
+			(at 26.67 69.8499 0)
 			(show_name no)
 			(do_not_autoplace no)
@@
 		)
 		(property "Value" "LM35CZ_TO92"
-			(at 50.8 67.31 0)
+			(at 55.88 67.31 0)
 			(hide yes)
 			(show_name no)
@@
 		)
 		(property "Footprint" "VAMK_IC:TO-92"
-			(at 50.8 69.85 0)
+			(at 55.88 69.85 0)
 			(hide yes)
 			(show_name no)
@@
 		)
 		(property "Datasheet" "\"\""
-			(at 50.8 72.39 0)
+			(at 55.88 72.39 0)
 			(hide yes)
 			(show_name no)
@@
 		)
 		(property "Description" "Analog Thermometer (-40°C to +110°C)"
-			(at 30.48 69.85 0)
+			(at 35.56 69.85 0)
 			(hide yes)
 			(show_name no)
@@
 		)
 		(property "Order Number Elfa" "73-088-10"
-			(at 50.8 74.93 0)
+			(at 55.88 74.93 0)
 			(hide yes)
 			(show_name no)
@@
 	(symbol
 		(lib_id "power:+12V")
-		(at 30.48 62.23 0)
+		(at 35.56 62.23 0)
 		(unit 1)
 		(body_style 1)
@@
 		(fields_autoplaced yes)
 		(property "Reference" "#PWR036"
-			(at 30.48 66.04 0)
+			(at 35.56 66.04 0)
 			(hide yes)
 			(show_name no)
@@
 		)
 		(property "Value" "+12V"
-			(at 30.48 57.15 0)
+			(at 35.56 57.15 0)
 			(show_name no)
 			(do_not_autoplace no)
@@
 		)
 		(property "Footprint" ""
-			(at 30.48 62.23 0)
+			(at 35.56 62.23 0)
 			(hide yes)
 			(show_name no)
@@
 		)
 		(property "Datasheet" ""
-			(at 30.48 62.23 0)
+			(at 35.56 62.23 0)
 			(hide yes)
 			(show_name no)
@@
 		)
 		(property "Description" "Power symbol creates a global label with name \"+12V\""
-			(at 30.48 62.23 0)
+			(at 35.56 62.23 0)
 			(hide yes)
 			(show_name no)
