File: KiCad_proj/signaalinlahetin/signaalinlahetin.kicad_pcb (KiCad board)
At the start: 2 copper layers, 20 parts, among them U1 UA741, U2 UA741, U3 UA741

Commit message: signaalin lähetin kaikki osat paikoillaan, ei johtoja vedetty vielä
Parts:
- added BC547_1: BC547_TO92_0.1A, VAMK_ANA:TO-92, F.Cu at (62.5, 78.2)
- added C7: 100NF_50V_CER, VAMK_C_SMD:C1206, F.Cu at (51.3, 78.2)
- added C8: 100NF_50V_CER, VAMK_C_SMD:C1206, F.Cu at (47.2, 67.6)
- added C9: 100NF_50V_CER, VAMK_C_SMD:C1206, F.Cu at (54.9, 75.7)
- added R14: 100R, VAMK_R_SMD:1206, F.Cu at (56.4, 78.2)
- added R15: 150R, VAMK_R_SMD:1206, F.Cu at (62.5, 81.3)
- added R3: 150k, VAMK_R_SMD:1206, F.Cu at (43.7, 73.2)
- added R4: 150k, VAMK_R_SMD:1206, F.Cu at (55.4, 72.1)
- added R5: 150k, VAMK_R_SMD:1206, F.Cu at (51.3, 81.3)
- added R6: 150k, VAMK_R_SMD:1206, F.Cu at (56.9, 81.3)
- added TM_BLOCK/2P1: TM_BLOCK_2P, VAMK_CON:TM_BLOCK_2P, F.Cu at (70.1, 80.8)
- added TM_BLOCK/3P1: TM_BLOCK_3P, VAMK_CON:TM_BLOCK_3P, F.Cu at (19.3, 66.0)
- added U4: UA741, VAMK_IC_SMD:SO8IC, F.Cu at (49.3, 73.2)
- C1, C2, C3, C4, C5, C6: footprint VAMK_C:C5_0 -> VAMK_C_SMD:C1206
- moved POTENTIO_M/1K_LIN1 132.8 mm to (69.1, 95.6), turned to -90 degrees
- moved U3 83.5 mm to (48.3, 86.4), turned to 90 degrees
- moved U2 75.4 mm to (38.6, 80.8), turned to 90 degrees
- moved R7 74.9 mm to (53.8, 85.9), turned to 180 degrees
- moved C4 70.5 mm to (53.8, 88.9), turned to 180 degrees
- moved R10 69.5 mm to (39.9, 73.2), turned to -90 degrees
- moved R13 69.0 mm to (41.1, 86.4), turned to 180 degrees
- moved C5 67.7 mm to (47.2, 80.3), turned to -90 degrees
- moved R12 66.5 mm to (41.1, 88.9)
- moved R9 64.6 mm to (36.1, 73.1), turned to -90 degrees
- moved U1 62.0 mm to (26.4, 80.8), turned to 90 degrees
- moved C2 60.2 mm to (43.2, 81.8), turned to -90 degrees
- moved R8 60.1 mm to (32.8, 73.1), turned to 90 degrees
- moved R11 60.0 mm to (35.6, 88.9)
- moved R2 56.2 mm to (35.6, 86.4)
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Connections:
- LM35CZ1 pad 1: unconnected-(LM35CZ1-+VS-Pad1) -> +12V
- POTENTIO_M/1K_LIN1 pad 3: Net-(POTENTIO_M/1K_LIN1-~-Pad3) -> GND
- R11 pad 1: Net-(POTENTIO_M/1K_LIN1-~-Pad3) -> GND
- R8 pad 2: Net-(R10-~-Pad1) -> Net-(R8-~-Pad2)
- R9 pad 1: Net-(R10-~-Pad1) -> Net-(R8-~-Pad2)
Other:
- board outline added: 60 x 50 mm

Commit message: signaalin lähetin, johdot vedetty paitsi virrat
Parts:
- moved R11 5.61 mm to (41.1, 89.4), turned to 180 degrees
- moved R12 5.61 mm to (35.6, 89.4), turned to 180 degrees
- moved R13 5.59 mm to (35.6, 86.4), turned to 0 degrees
- moved R2 5.59 mm to (41.1, 86.4), turned to 180 degrees
- moved C9 1.61 mm to (55.4, 74.2)
- moved R4 0.51 mm to (55.4, 71.6)
- turned R5 to 180 degrees
Routing:
- net Net-(U3-+): track 0.00 -> 43.2 mm
- net Net-(TM_BLOCK/2P1-Pin_1): track 0.00 -> 28.3 mm
- net +12V: track 0.00 -> 22.7 mm
- net Net-(U4-~): track 0.00 -> 17.1 mm
- net Net-(U4-+): track 0.00 -> 14.3 mm
- net Net-(U2--): track 0.00 -> 13.9 mm
- net Net-(BC547_1-B): track 0.00 -> 12.7 mm
- net Net-(U3--): track 0.00 -> 12.0 mm
- net Net-(U1--): track 0.00 -> 11.2 mm
- net -12V: track 0.00 -> 10.4 mm
- net Net-(LM35CZ1-Vout): track 0.00 -> 10.1 mm
- net Net-(U4--): track 0.00 -> 9.89 mm
- net Net-(BC547_1-C): track 0.00 -> 9.56 mm
- net Net-(U2-~): track 0.00 -> 7.66 mm
- net Net-(BC547_1-E): track 0.00 -> 6.23 mm
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